File: TeensyRF.brd (EAGLE design)
At the start: 40 x 40 mm, 23 parts, among them X1 SMA-142-0701-801/806, X2 SMA-142-0701-801/806, X3 SMA-142-0701-801/806, X4 SMA-142-0701-801/806

Commit message: Fixed R11 R12 mixup
Parts:
- R11: value 1.5k -> 2k
- R12: value 2k -> 1.5k
Changed lines of the file:
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@@
 <layer number="59" name="tCarbon" color="7" fill="1" visible="no" active="no"/>
 <layer number="60" name="bCarbon" color="7" fill="1" visible="no" active="no"/>
-<layer number="90" name="Modules" color="5" fill="1" visible="yes" active="yes"/>
+<layer number="90" name="Modules" color="5" fill="1" visible="no" active="no"/>
 <layer number="91" name="Nets" color="2" fill="1" visible="no" active="no"/>
 <layer number="92" name="Busses" color="1" fill="1" visible="no" active="no"/>
@@
 <attribute name="NAME" x="29.538" y="7.9255" size="0.4064" layer="25"/>
 </element>
-<element name="R11" library="SparkFun-Resistors" package="0805" value="1.5k" x="35.5" y="32.6" smashed="yes">
+<element name="R11" library="SparkFun-Resistors" package="0805" value="2k" x="35.5" y="32.6" smashed="yes">
 <attribute name="NAME" x="34.738" y="33.4255" size="0.4064" layer="25"/>
 </element>
-<element name="R12" library="SparkFun-Resistors" package="0805" value="2k" x="35.5" y="30.4" smashed="yes" rot="R180">
+<element name="R12" library="SparkFun-Resistors" package="0805" value="1.5k" x="35.5" y="30.4" smashed="yes" rot="R180">
 <attribute name="NAME" x="33.962" y="30.4745" size="0.4064" layer="25" rot="R180"/>
 </element>
